File: board/OpAmp.kicad_sch (KiCad schematic)
At the start: 15 parts, among them U3 Opamp_Dual, U8 Opamp_Dual

Commit message: Add Mega_Fits, Add Verticle Connectors, Add TFT GND & 5V, Changed Buzzer to pin 11, Fix Mosfet Footprint, Remove I2C
Parts:
- Conn4: footprint MRDT_Connectors:MOLEX_SL_04_Horizontal -> MRDT_Connectors:MOLEX_SL_04_Vertical
Changed lines of the file:
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@@
 			)
 		)
-		(property "Footprint" "MRDT_Connectors:MOLEX_SL_04_Horizontal"
+		(property "Footprint" "MRDT_Connectors:MOLEX_SL_04_Vertical"
 			(at 50.8 38.1 0)
 			(effects
